Commit message: add proper urdf

File: example/robot.urdf (robot description, URDF)
Before this commit: robot panda, 41 links, 40 joints
Links:
- removed link camera_bottom_screw_frame
- removed link camera_color_frame
- removed link camera_color_optical_frame
- removed link camera_depth_frame
- removed link camera_depth_optical_frame
- removed link camera_infra1_frame
- removed link camera_infra1_optical_frame
- removed link camera_infra2_frame
- removed link camera_infra2_optical_frame
- removed link camera_link
- removed link panda1_box
- removed link panda_camera_support_link
- removed link panda_hand
- removed link panda_hand_sc
- removed link panda_hand_tcp
- removed link panda_leftfinger
- removed link panda_ref_camera_link
- removed link panda_rightfinger
- removed link pedestal
- removed link support_link
- removed link wall_link_1
- removed link wall_link_2
- removed link wall_link_3
- added link box; collision box size=0.1 0.1 0.2; visual box size=0.1 0.1 0.2
- added link foot, mass 0.9; visual mesh filename=package://panda_torque_mpc/meshes/meshes_panda_human/foot_m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 scale=0.0060 0.0060 0.0060; visual mesh filename=package://panda_torque_mpc/meshes/meshes_panda_human/foot_m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 scale=0.0060 0.0060 0.0060
- added link hand, mass 0.45; visual mesh filename=package://panda_torque_mpc/meshes/meshes_panda_human/hand_m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 scale=0.0060 0.0060 0.0060; visual mesh filename=package://panda_torque_mpc/meshes/meshes_panda_human/hand_m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 scale=0.0060 0.0060 0.0060
- added link lowerarm, mass 1.28; visual mesh filename=package://panda_torque_mpc/meshes/meshes_panda_human/elbow_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 scale=0.0055 0.0055 0.0055; visual mesh filename=package://panda_torque_mpc/meshes/meshes_panda_human/elbow_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 scale=0.0055 0.0055 0.0055
- added link lowerleg, mass 3.6; visual mesh filename=package://panda_torque_mpc/meshes/meshes_panda_human/lowerl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 scale=0.0063 0.0065 0.007; visual mesh filename=package://panda_torque_mpc/meshes/meshes_panda_human/lowerl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 scale=0.0063 0.0065 0.007
- added link trunk, mass 35.47; visual mesh filename=package://panda_torque_mpc/meshes/meshes_panda_human/abdome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 scale=0.0055 0.0055 0.0055; visual mesh filename=package://panda_torque_mpc/meshes/meshes_panda_human/head_m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 scale=0.0055 0.0055 0.0055
- added link upperarm, mass 1.8; visual mesh filename=package://panda_torque_mpc/meshes/meshes_panda_human/should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 scale=0.0055 0.0055 0.0055; visual mesh filename=package://panda_torque_mpc/meshes/meshes_panda_human/should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 scale=0.0055 0.0055 0.0055
- added link upperleg, mass 9.22; visual mesh filename=package://panda_torque_mpc/meshes/meshes_panda_human/knee_m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 scale=0.006 0.006 0.006; visual mesh filename=package://panda_torque_mpc/meshes/meshes_panda_human/knee_m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 scale=0.006 0.006 0.006
- link panda_link0: geometry collision mesh filename=package://franka_description/meshes/collision/link0.stl; visual mesh filename=package://franka_description/meshes/visual/link0.dae
- link panda_link0_sc: geometry 
- link panda_link1: geometry collision mesh filename=package://franka_description/meshes/collision/link1.stl; visual mesh filename=package://franka_description/meshes/visual/link1.dae
- link panda_link1_sc: geometry 
- link panda_link2: geometry collision mesh filename=package://franka_description/meshes/collision/link2.stl; visual mesh filename=package://franka_description/meshes/visual/link2.dae
- link panda_link2_sc: geometry 
- link panda_link3: geometry collision mesh filename=package://franka_description/meshes/collision/link3.stl; visual mesh filename=package://franka_description/meshes/visual/link3.dae
- link panda_link3_sc: geometry 
- link panda_link4: geometry collision mesh filename=package://franka_description/meshes/collision/link4.stl; visual mesh filename=package://franka_description/meshes/visual/link4.dae
- link panda_link4_sc: geometry 
- link panda_link5: geometry collision mesh filename=package://franka_description/meshes/collision/link5.stl; visual mesh filename=package://franka_description/meshes/visual/link5.dae
- link panda_link5_sc: geometry 
- link panda_link6: geometry collision mesh filename=package://franka_description/meshes/collision/link6.stl; visual mesh filename=package://franka_description/meshes/visual/link6.dae
- link panda_link6_sc: geometry 
- link panda_link7: geometry collision mesh filename=package://franka_description/meshes/collision/link7.stl; visual mesh filename=package://franka_description/meshes/visual/link7.dae
- link panda_link7_sc: geometry 
- link panda_link8: mass 0 -> None
Joints:
- removed joint camera_color_joint
- removed joint camera_color_optical_joint
- removed joint camera_depth_joint
- removed joint camera_depth_optical_joint
- removed joint camera_infra1_joint
- removed joint camera_infra1_optical_joint
- removed joint camera_infra2_joint
- removed joint camera_infra2_optical_joint
- removed joint camera_joint
- removed joint camera_link_joint
- removed joint panda1_box_joint
- removed joint panda_camera_support_joint
- removed joint panda_finger_joint1
- removed joint panda_finger_joint2
- removed joint panda_hand_joint
- removed joint panda_hand_sc_joint
- removed joint panda_hand_tcp_joint
- removed joint panda_ref_camera_joint
- removed joint pedestal_joint
- removed joint support_joint
- removed joint wall_joint_1
- removed joint wall_joint_2
- removed joint wall_joint_3
- removed joint world_joint
- added joint ankle_Z: type revolute, parent foot, child lowerleg, origin xyz=0.0 0.0 0.0 rpy=0 0 0, axis 0 0 1, limit lower=-0.785398 upper=3.14159 effort=500.0 velocity=200.0
- added joint elbow_Z: type revolute, parent upperarm, child lowerarm, origin xyz=0.262 0.0 0.0 rpy=0 0 0, axis 0 0 1, limit lower=0 upper=2.74889 effort=500.0 velocity=200.0
- added joint flange_to_box: type fixed, parent panda_link8, child box, origin xyz=0 0 0.1 rpy=0 -0 0, axis 0 0 1
- added joint hand_fixed: type fixed, parent lowerarm, child hand, origin xyz=0.273 0.0 0.0 rpy=0 0 0, axis 0 0 1, limit lower=-1.5708 upper=1.5708 effort=500.0 velocity=200.0
- added joint knee_Z: type revolute, parent lowerleg, child upperleg, origin xyz=0.418 0.0 0.0 rpy=0 0 0, axis 0 0 1, limit lower=-2.74889 upper=2.74889 effort=500.0 velocity=200.0
- added joint lumbar_Z: type revolute, parent upperleg, child trunk, origin xyz=0.417 0.0 0.0 rpy=0 0 0, axis 0 0 1, limit lower=-3.14 upper=0 effort=500.0 velocity=200.0
- added joint shoulder_Z: type revolute, parent trunk, child upperarm, origin xyz=0.46 0.0 0.0 rpy=0 0 0, axis 0 0 1, limit lower=-3.14 upper=1.54 effort=500.0 velocity=200.0
- added joint world_to_human: type fixed, parent world, child foot, origin xyz=0. 0. 0. rpy=1.57 -0 -1.57, axis 0 0 1
- added joint world_to_panda: type fixed, parent world, child panda_link0, origin xyz=0.8 0 0.8 rpy=0 -0 0, axis 0 0 1
